Commit message: Changes for iit-relax repo

File: mir_description/urdf/include/sick_s300.urdf.xacro (robot description, xacro)
@@ -5,5 +5,5 @@
   <xacro:property name="laser_y" value="0.155" />
   <xacro:property name="laser_z" value="0.185" />
-  <xacro:property name="laser_mass" value="2.0" />
+  <xacro:property name="laser_mass" value="1.2" />
   <xacro:macro name="sick_s300" params="link topic prefix">
     <link name="${prefix}${link}">

File: mir_description/urdf/mir.urdf.xacro (robot description, xacro)
@@ -1,7 +1,7 @@
 <?xml version="1.0"?>
 <robot xmlns:xacro="http://ros.org/wiki/xacro"
-       name="mir_250" >
-  <!-- MiR100 base -->
-  <xacro:include filename="$(find mir_description)/urdf/include/mir_250_v1.urdf.xacro" />
+       name="mir" >
+  <!-- MiR base -->
+  <xacro:include filename="$(find mir_description)/urdf/include/mir_v1.urdf.xacro" />
   <xacro:include filename="$(find mir_description)/urdf/include/common.gazebo.xacro" />
   <xacro:arg name="tf_prefix" default="" />
@@ -13,5 +13,5 @@
     <xacro:property name="prefix" value="${tf_prefix_}/" />
   </xacro:unless>
-  <xacro:mir_250 prefix="${prefix}"/>
+  <xacro:mir prefix="${prefix}" />
   <xacro:controller_plugin_gazebo robot_namespace=""/>
   <!-- instead of the controller_plugin_gazebo, you can use the diffdrive controller like this:
@@ -19,6 +19,6 @@
       left_wheel_joint="left_wheel_joint"
       right_wheel_joint="right_wheel_joint"
-      wheel_separation="${2*mir_250_act_wheel_dy}"
-      wheel_radius="${mir_250_act_wheel_radius}"/>
+      wheel_separation="${2*mir_act_wheel_dy}"
+      wheel_radius="${mir_act_wheel_radius}"/>
   -->
 </robot>
